File: usb.kicad_sch (KiCad schematic)
At the start: 26 parts, among them J1 USB_A, J2 USB_A, J4 USB_C_Receptacle_USB2.0, U1 FE1.1s, U3 SRV05-4, U4 SRV05-4, U6 AP2552W6, Y1 12MHz

Commit message: fix some erc/drc
Changed lines of the file:
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@@
+    (stroke (width 0) (type default))
+  )
+  (wire (pts (xy 71.12 63.5) (xy 81.28 63.5))
     (stroke (width 0) (type default))
   )
@@
         )
       )
+    )
+  )
+  (symbol (lib_id "power:PWR_FLAG") (at 81.28 63.5 0) (unit 1)
+    (in_bom yes) (on_board yes) (dnp no) (fields_autoplaced)
+    (property "Reference" "#FLG03" (at 81.28 61.595 0)
+      (effects (font (size 1.27 1.27)) hide)
+    )
+    (property "Value" "PWR_FLAG" (at 81.28 58.42 0)
+      (effects (font (size 1.27 1.27)))
+    )
+    (property "Footprint" "" (at 81.28 63.5 0)
+      (effects (font (size 1.27 1.27)) hide)
+    )
+    (property "Datasheet" "~" (at 81.28 63.5 0)
+      (effects (font (size 1.27 1.27)) hide)
+    )
+    (pin "1")
+    (instances
+      (project "das-kb4-bara2"
+        (path "/d0e4eaec-96cb-4a0e-a384-5b3e3f5f8d5d/f457a5c4-270e-459d-a4f0-150cf90e3909"
+          (reference "#FLG03") (unit 1)
+        )
+      )
