File: hw/r2023-12/das-kb4-bara2.kicad_sch (KiCad schematic)
At the start: 6 parts, among them U5 XC6206PxxxMR

Commit message: r2023-12: add more gnd pins
Parts:
- TP1, TP2, TP3: now left out of the parts list
Changed lines of the file:
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@@
   )
   (symbol (lib_id "Connector:TestPoint") (at 58.42 111.76 180) (unit 1)
-    (in_bom yes) (on_board yes) (dnp no) (fields_autoplaced)
+    (in_bom no) (on_board yes) (dnp no) (fields_autoplaced)
     (property "Reference" "TP2" (at 60.96 113.792 0)
       (effects (font (size 1.27 1.27)) (justify right))
@@
   )
   (symbol (lib_id "Connector:TestPoint") (at 43.18 111.76 180) (unit 1)
-    (in_bom yes) (on_board yes) (dnp no) (fields_autoplaced)
+    (in_bom no) (on_board yes) (dnp no) (fields_autoplaced)
     (property "Reference" "TP1" (at 45.72 113.792 0)
       (effects (font (size 1.27 1.27)) (justify right))
@@
   )
   (symbol (lib_id "Connector:TestPoint") (at 73.66 116.84 0) (unit 1)
-    (in_bom yes) (on_board yes) (dnp no) (fields_autoplaced)
+    (in_bom no) (on_board yes) (dnp no) (fields_autoplaced)
     (property "Reference" "TP3" (at 76.2 112.268 0)
       (effects (font (size 1.27 1.27)) (justify left))
