File: hw/r2023-12/keys_mcu.kicad_sch (KiCad schematic)
At the start: 28 parts, among them J3 Conn_01x26_Socket, J5 Conn_ARM_JTAG_SWD_10, J6 Conn_01x06_Socket, SW1 PWR, SW2 MUTE, SW2 Volume, SW3 PREV, SW4 PLAY_PAUSE, SW5 NEXT, U2 STM32G431CBUx

Commit message: r2023-12: add more gnd pins
Parts:
- added JP2: Jumper_2_Open, Connector_PinHeader_2.54mm:PinHeader_1x02_P2.54mm_Vertical, symbol Jumper:Jumper_2_Open
Connections:
- net GND: now also JP2.1 (A), JP2.2 (B)
Changed lines of the file:
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@@
   (junction (at 142.24 25.4) (diameter 0) (color 0 0 0 0)
+  )
+  (junction (at 154.94 177.8) (diameter 0) (color 0 0 0 0)
   )
   (junction (at 139.7 48.26) (diameter 0) (color 0 0 0 0)
@@
     (stroke (width 0) (type default))
   )
+  (wire (pts (xy 165.1 177.8) (xy 154.94 177.8))
+    (stroke (width 0) (type default))
+  )
   (wire (pts (xy 142.24 48.26) (xy 142.24 55.88))
     (stroke (width 0) (type default))
@@
     (stroke (width 0) (type default))
   )
+  (wire (pts (xy 154.94 172.72) (xy 154.94 177.8))
+    (stroke (width 0) (type default))
+  )
   (wire (pts (xy 157.48 91.44) (xy 162.56 91.44))
     (stroke (width 0) (type default))
@@
   )
   (wire (pts (xy 228.6 48.26) (xy 223.52 48.26))
+    (stroke (width 0) (type default))
+  )
+  (wire (pts (xy 165.1 172.72) (xy 165.1 177.8))
     (stroke (width 0) (type default))
   )
@@
         (path "/d0e4eaec-96cb-4a0e-a384-5b3e3f5f8d5d/7c81bc9d-f306-4c7f-90ce-10f7b22818e4"
           (reference "R5") (unit 1)
+        )
+      )
+    )
+  )
+  (symbol (lib_id "power:GND") (at 154.94 177.8 0) (unit 1)
+    (in_bom yes) (on_board yes) (dnp no) (fields_autoplaced)
+    (property "Reference" "#PWR056" (at 154.94 184.15 0)
+      (effects (font (size 1.27 1.27)) hide)
+    )
+    (property "Value" "GND" (at 154.94 182.88 0)
+      (effects (font (size 1.27 1.27)))
+    )
+    (property "Footprint" "" (at 154.94 177.8 0)
+      (effects (font (size 1.27 1.27)) hide)
+    )
+    (property "Datasheet" "" (at 154.94 177.8 0)
+      (effects (font (size 1.27 1.27)) hide)
+    )
+    (pin "1")
+    (instances
+      (project "das-kb4-bara2"
+        (path "/d0e4eaec-96cb-4a0e-a384-5b3e3f5f8d5d/7c81bc9d-f306-4c7f-90ce-10f7b22818e4"
+          (reference "#PWR056") (unit 1)
         )
       )
@@
         )
       )
+    )
+  )
+  (symbol (lib_id "Jumper:Jumper_2_Open") (at 160.02 172.72 180) (unit 1)
+    (in_bom yes) (on_board yes) (dnp no) (fields_autoplaced)
+    (property "Reference" "JP2" (at 160.02 167.64 0)
+      (effects (font (size 1.27 1.27)))
+    )
+    (property "Value" "Jumper_2_Open" (at 160.02 170.18 0)
+      (effects (font (size 1.27 1.27)))
+    )
+    (property "Footprint" "Connector_PinHeader_2.54mm:PinHeader_1x02_P2.54mm_Vertical" (at 160.02 172.72 0)
+      (effects (font (size 1.27 1.27)) hide)
+    )
+    (property "Datasheet" "~" (at 160.02 172.72 0)
+      (effects (font (size 1.27 1.27)) hide)
+    )
+    (pin "1")
+    (pin "2")
+    (instances
+      (project "das-kb4-bara2"
+        (path "/d0e4eaec-96cb-4a0e-a384-5b3e3f5f8d5d/a2d5569b-3e38-48fc-9c53-ff19306ffa54"
+          (reference "JP2") (unit 1)
+        )
+        (path "/d0e4eaec-96cb-4a0e-a384-5b3e3f5f8d5d/7c81bc9d-f306-4c7f-90ce-10f7b22818e4"
+          (reference "JP3") (unit 1)
+        )
+      )
