File: hw/r2023-12/usb.kicad_sch (KiCad schematic)
At the start: 26 parts, among them J1 USB_A, J2 USB_A, J4 USB_C_Receptacle_USB2.0, U1 FE1.1s, U3 SRV05-4, U4 SRV05-4, U6 AP2552W6, Y1 12MHz

Commit message: r2023-12: add more gnd pins
Parts:
- TP2: now left out of the parts list
Changed lines of the file:
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@@
   )
   (symbol (lib_id "Connector:TestPoint") (at 99.06 111.76 90) (unit 1)
-    (in_bom yes) (on_board yes) (dnp no) (fields_autoplaced)
+    (in_bom no) (on_board yes) (dnp no) (fields_autoplaced)
     (property "Reference" "TP2" (at 95.758 106.68 90)
       (effects (font (size 1.27 1.27)))
