File: hw/r2023-12/usb.kicad_sch (KiCad schematic)
At the start: 26 parts, among them J1 USB_A, J2 USB_A, J4 USB_C_Receptacle_USB2.0, U1 FE1.1s, U3 SRV05-4, U4 SRV05-4, U6 AP2552W6, Y1 12MHz

Commit message: r2023_12: add firmware notes and comments on matrix decode
No intentional changes, just text added while working out the firmware.
Parts:
- renumbered TP2 to TP4
Changed lines of the file:
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@@
     (instances
       (project "das-kb4-bara2"
-        (path "/d0e4eaec-96cb-4a0e-a384-5b3e3f5f8d5d"
-          (reference "J2") (unit 1)
-        )
         (path "/d0e4eaec-96cb-4a0e-a384-5b3e3f5f8d5d/f457a5c4-270e-459d-a4f0-150cf90e3909"
           (reference "J2") (unit 1)
@@
   (symbol (lib_id "Connector:TestPoint") (at 99.06 111.76 90) (unit 1)
     (in_bom no) (on_board yes) (dnp no) (fields_autoplaced)
-    (property "Reference" "TP2" (at 95.758 106.68 90)
+    (property "Reference" "TP4" (at 95.758 106.68 90)
       (effects (font (size 1.27 1.27)))
     )
@@
     (instances
       (project "das-kb4-bara2"
-        (path "/d0e4eaec-96cb-4a0e-a384-5b3e3f5f8d5d"
-          (reference "TP2") (unit 1)
-        )
         (path "/d0e4eaec-96cb-4a0e-a384-5b3e3f5f8d5d/f457a5c4-270e-459d-a4f0-150cf90e3909"
           (reference "TP4") (unit 1)
@@
     (instances
       (project "das-kb4-bara2"
-        (path "/d0e4eaec-96cb-4a0e-a384-5b3e3f5f8d5d"
-          (reference "Y1") (unit 1)
-        )
         (path "/d0e4eaec-96cb-4a0e-a384-5b3e3f5f8d5d/f457a5c4-270e-459d-a4f0-150cf90e3909"
           (reference "Y1") (unit 1)
@@
     (instances
       (project "das-kb4-bara2"
-        (path "/d0e4eaec-96cb-4a0e-a384-5b3e3f5f8d5d"
-          (reference "U1") (unit 1)
-        )
         (path "/d0e4eaec-96cb-4a0e-a384-5b3e3f5f8d5d/f457a5c4-270e-459d-a4f0-150cf90e3909"
           (reference "U1") (unit 1)
@@
     (instances
       (project "das-kb4-bara2"
-        (path "/d0e4eaec-96cb-4a0e-a384-5b3e3f5f8d5d"
+        (path "/d0e4eaec-96cb-4a0e-a384-5b3e3f5f8d5d/f457a5c4-270e-459d-a4f0-150cf90e3909"
           (reference "J1") (unit 1)
-        )
-        (path "/d0e4eaec-96cb-4a0e-a384-5b3e3f5f8d5d/f457a5c4-270e-459d-a4f0-150cf90e3909"
-          (reference "J1") (unit 1)
